Commit message: Add gazebo

File: src/ugv_main/ugv_description/urdf/ugv_beast.ros2_control.xacro (robot description, xacro)
@@ -4,9 +4,9 @@
     ros2_control system block for the UGV beast.
     Real robot  -> ugv_hardware/UgvSystemHardware (owns the ESP32 UART).
-    use_sim=true -> gazebo_ros2_control GazeboSystem. This branch is a FUTURE HOOK:
-    the Gazebo Classic sim still runs on the legacy planar_move plugin today, and true
-    sim parity is deferred to the Jazzy / new-Gazebo upgrade. Keeping the branch here
-    means the upgrade only has to swap this one <plugin> (the controller YAML and the
-    interface declarations below carry over unchanged).
+    use_sim=true -> gz_ros2_control GazeboSimSystem (new Gazebo / Harmonic). The same
+    diff_drive_controller + broadcaster config (ugv_beast_controllers.yaml) and the
+    interface declarations below carry over unchanged between real and sim — only this
+    one <plugin> differs. The gz sensors and the gz_ros2_control system plugin itself
+    are contributed by ugv_beast.gazebo.xacro (also gated on use_sim).
   -->
   <xacro:macro name="ugv_ros2_control"
@@ -18,5 +18,5 @@
       <hardware>
         <xacro:if value="${use_sim}">
-          <plugin>gazebo_ros2_control/GazeboSystem</plugin>
+          <plugin>gz_ros2_control/GazeboSimSystem</plugin>
         </xacro:if>
         <xacro:unless value="${use_sim}">

File: src/ugv_main/ugv_description/urdf/ugv_beast.urdf.xacro (robot description, xacro)
@@ -3,11 +3,18 @@
   name="ugv_beast"
   xmlns:xacro="http://www.ros.org/wiki/xacro">
-  <!-- ros2_control: real robot by default; use_sim is a future hook (see the macro). -->
+  <!-- ros2_control: real robot by default; use_sim swaps in gz_ros2_control. -->
   <xacro:arg name="use_sim" default="false"/>
   <xacro:arg name="serial_device" default="/dev/ttyAMA0"/>
+  <xacro:arg name="controllers_file"
+             default="$(find ugv_bringup)/config/ugv_beast_controllers.yaml"/>
   <xacro:include filename="$(find ugv_description)/urdf/ugv_beast.ros2_control.xacro"/>
   <xacro:ugv_ros2_control name="ugv_beast"
                           use_sim="$(arg use_sim)"
                           serial_device="$(arg serial_device)"/>
+  <!-- new-Gazebo sensors + gz_ros2_control system + track friction (sim only). -->
+  <xacro:if value="$(arg use_sim)">
+    <xacro:include filename="$(find ugv_description)/urdf/ugv_beast.gazebo.xacro"/>
+    <xacro:ugv_beast_gazebo controllers_yaml="$(arg controllers_file)"/>
+  </xacro:if>
   <link name="base_footprint"></link>
   <link
@@ -71,12 +78,12 @@
         rpy="0 0 0" />
       <mass
-        value="0.0602574557338752" />
-      <inertia
-        ixx="1.41463499717618E-05"
-        ixy="5.40675906873518E-18"
-        ixz="2.24533090468138E-31"
-        iyy="1.86414633348696E-05"
-        iyz="1.86664834767948E-19"
-        izz="1.41463499717618E-05" />
+        value="0.207085933743005" />
+      <inertia
+        ixx="0.000116541923504163"
+        ixy="0"
+        ixz="0"
+        iyy="0.000170742352371108"
+        iyz="0"
+        izz="0.000116541923504163" />
     </inertial>
     <visual>
@@ -94,11 +101,12 @@
       </material>
     </visual>
-    <collision>
-      <origin
-        xyz="0 0 0"
-        rpy="0 0 0" />
-      <geometry>
-        <mesh
-          filename="package://ugv_description/meshes/ugv_beast/left_up_wheel_link.stl" />
+    <!-- Sim contact: cylinder (radius = controller wheel_radius) instead of the
+         mesh; the mesh stays as the visual. Axis along the axle (y) via roll=pi/2. -->
+    <collision>
+      <origin
+        xyz="0 0.0155 0"
+        rpy="1.5708 0 0" />
+      <geometry>
+        <cylinder radius="0.025" length="0.03"/>
       </geometry>
     </collision>
@@ -124,12 +132,12 @@
         rpy="0 0 0" />
       <mass
-        value="0.00565722297095184" />
-      <inertia
-        ixx="2.80120931171082E-07"
-        ixy="1.73012571052522E-19"
-        ixz="7.08181663938282E-33"
-        iyy="4.2446851103923E-07"
-        iyz="5.90904673131262E-21"
-        izz="2.80120931171082E-07" />
+        value="0.207085933743005" />
+      <inertia
+        ixx="0.000116541923504163"
+        ixy="0"
+        ixz="0"
+        iyy="0.000170742352371108"
+        iyz="0"
+        izz="0.000116541923504163" />
     </inertial>
     <visual>
@@ -149,9 +157,8 @@
     <collision>
       <origin
-        xyz="0 0 0"
-        rpy="0 0 0" />
-      <geometry>
-        <mesh
-          filename="package://ugv_description/meshes/ugv_beast/left_down_wheel_link.stl" />
+        xyz="0 0.006 0"
+        rpy="1.5708 0 0" />
+      <geometry>
+        <cylinder radius="0.025" length="0.03"/>
       </geometry>
     </collision>
@@ -177,12 +184,12 @@
         rpy="0 0 0" />
       <mass
-        value="0.0602574557338752" />
-      <inertia
-        ixx="1.41463499717618E-05"
-        ixy="-5.34398065104604E-18"
-        ixz="2.21929095291762E-31"
-        iyy="1.86414633348696E-05"
-        iyz="-1.86664834767948E-19"
-        izz="1.41463499717618E-05" />
+        value="0.207085933743005" />
+      <inertia
+        ixx="0.000116541923504163"
+        ixy="0"
+        ixz="0"
+        iyy="0.000170742352371108"
+        iyz="0"
+        izz="0.000116541923504163" />
     </inertial>
     <visual>
@@ -202,9 +209,8 @@
     <collision>
       <origin
-        xyz="0 0 0"
-        rpy="0 0 0" />
-      <geometry>
-        <mesh
-          filename="package://ugv_description/meshes/ugv_beast/right_up_wheel_link.stl" />
+        xyz="0 -0.0155 0"
+        rpy="1.5708 0 0" />
+      <geometry>
+        <cylinder radius="0.025" length="0.03"/>
       </geometry>
     </collision>
@@ -230,12 +236,12 @@
         rpy="0 0 0" />
       <mass
-        value="0.00565722297095184" />
-      <inertia
-        ixx="2.80120931171082E-07"
-        ixy="-1.70986035603665E-19"
-        ixz="6.99903667727259E-33"
-        iyy="4.2446851103923E-07"
-        iyz="-5.90904673131262E-21"
-        izz="2.80120931171082E-07" />
+        value="0.207085933743005" />
+      <inertia
+        ixx="0.000116541923504163"
+        ixy="0"
+        ixz="0"
+        iyy="0.000170742352371108"
+        iyz="0"
+        izz="0.000116541923504163" />
     </inertial>
     <visual>
@@ -255,9 +261,8 @@
     <collision>
       <origin
-        xyz="0 0 0"
-        rpy="0 0 0" />
-      <geometry>
-        <mesh
-          filename="package://ugv_description/meshes/ugv_beast/right_down_wheel_link.stl" />
+        xyz="0 -0.006 0"
+        rpy="1.5708 0 0" />
+      <geometry>
+        <cylinder radius="0.025" length="0.03"/>
       </geometry>
     </collision>
